File: pcb/mks_mkb1/mks_mkb1.kicad_pcb (KiCad board)
At the start: 2 copper layers, 272 parts, among them J1 Conn_01x02, J2 Conn_01x02, J3 Conn_01x06_Pin, J4 Conn_01x06_Pin, SW1 SW_Push, SW10 SW_Push, SW11 SW_Push, SW12 SW_Push, SW13 SW_Push, SW14 SW_Push, SW15 SW_Push, SW16 SW_Push, SW17 SW_Push, SW18 SW_Push, SW19 SW_Push, SW2 SW_Push, SW20 SW_Push, SW21 SW_Push, SW22 SW_Push, SW23 SW_Push, SW24 SW_Push, SW25 SW_Push, SW26 SW_Push, SW27 SW_Push, SW28 SW_Push, SW29 SW_Push, SW3 SW_Push, SW30 SW_Push, SW31 SW_Push, SW32 SW_Push, SW33 SW_Push, SW34 SW_Push, SW35 SW_Push, SW36 SW_Push, SW37 SW_Push, SW38 SW_Push, SW39 SW_Push, SW4 SW_Push, SW40 SW_Push, SW41 SW_Push, SW42 SW_Push, SW43 SW_Push, SW44 SW_Push, SW45 SW_Push, SW46 SW_Push, SW47 SW_Push, SW48 SW_Push, SW49 SW_Push, SW5 SW_Push, SW50 SW_Push, SW51 SW_Push, SW52 SW_Push, SW53 SW_Push, SW54 SW_Push, SW55 SW_Push, SW56 SW_Push, SW57 SW_Push, SW58 SW_Push, SW59 SW_Push, SW6 SW_Push, SW60 SW_Push, SW61 SW_DP3T, SW62 SW_DP3T, SW7 SW_Push, SW8 SW_Push, SW9 SW_Push, U1 XIAO-nRF52840-SMD, U2 MT3608, U3 TPS2116DRL, U4 XIAO-nRF52840-SMD, U5 MT3608, U6 TPS2116DRL

Commit message: mod1
Parts:
- removed C_OUT3: 22uF, Capacitor_SMD:C_0805_2012Metric
- removed D100, D101, D102, D103, D104, D105, D106, D107, D108, D109, D110, D111, D112, D113, D114, D115, D116, D117, D118, D119, D120, D121, D122, D123, D124, D125, D126, D127, D128, D129, D130, D131, D132, D133, D134, D135, D136, D137, D138, D139, D140, D141, D142, D143, D144, D145, D146, D147, D148, D149, D150, D91, D92, D93, D94, D95, D96, D97, D98, D99: D, Diode_SMD:D_SOD-123
- removed R2, R5: 39kR, Resistor_SMD:R_0603_1608Metric
- removed R3, R6: 10kR, Resistor_SMD:R_0603_1608Metric
- added C_OUT1: 22uF, Capacitor_SMD:C_0805_2012Metric, F.Cu at (24.6, 127.0)
- added C_PM1: 4.7µF, Capacitor_SMD:C_0603_1608Metric, F.Cu at (88.8, 148.8)
- added C_PM2: 4.7µF, Capacitor_SMD:C_0603_1608Metric, F.Cu at (88.8, 151.3)
- added C_PM3: 47µF, Capacitor_SMD:C_0603_1608Metric, F.Cu at (100.0, 152.7)
- added C_PM4: 4.7µF, Capacitor_SMD:C_0603_1608Metric, F.Cu at (278.7, 158.8)
- added C_PM5: 4.7µF, Capacitor_SMD:C_0603_1608Metric, F.Cu at (276.7, 164.2)
- added C_PM6: 47µF, Capacitor_SMD:C_0603_1608Metric, F.Cu at (279.0, 169.5)
- added C_SR1: 0.1µF, Capacitor_SMD:C_0603_1608Metric, F.Cu at (93.7, 124.2)
- added C_SR2: 0.1µF, Capacitor_SMD:C_0603_1608Metric, F.Cu at (270.8, 159.5)
- added REF**: MountingHole_2.2mm_M2, MountingHole:MountingHole_2.2mm_M2, F.Cu at (140.0, 110.2)
- added REF**: MountingHole_2.2mm_M2, MountingHole:MountingHole_2.2mm_M2, F.Cu at (15.0, 110.2)
- added REF**: MountingHole_2.2mm_M2, MountingHole:MountingHole_2.2mm_M2, F.Cu at (140.0, 25.2)
- added REF**: MountingHole_2.2mm_M2, MountingHole:MountingHole_2.2mm_M2, F.Cu at (111.0, 150.2)
- added REF**: MountingHole_2.2mm_M2, MountingHole:MountingHole_2.2mm_M2, F.Cu at (15.0, 150.2)
- added REF**: MountingHole_2.2mm_M2, MountingHole:MountingHole_2.2mm_M2, F.Cu at (15.0, 25.2)
- added R_DM2: 10k, Resistor_SMD:R_0603_1608Metric, F.Cu at (94.0, 120.0)
- added R_DM4: 10k, Resistor_SMD:R_0603_1608Metric, F.Cu at (97.2, 123.0)
- added R_DM7: 10k, Resistor_SMD:R_0603_1608Metric, F.Cu at (257.2, 171.2)
- added R_DM8: 10k, Resistor_SMD:R_0603_1608Metric, F.Cu at (262.7, 176.0)
- added R_PM1: 30kR, Resistor_SMD:R_0603_1608Metric, F.Cu at (94.7, 147.2)
- added R_PM2: 10kR, Resistor_SMD:R_0603_1608Metric, F.Cu at (94.3, 152.8)
- added R_PM3: 30kR, Resistor_SMD:R_0603_1608Metric, F.Cu at (268.7, 171.2)
- added R_PM4: 10kR, Resistor_SMD:R_0603_1608Metric, F.Cu at (272.4, 176.0)
- added U7: 74HC595, Package_SO:SOIC-16_3.9x9.9mm_P1.27mm, F.Cu at (105.1, 121.5)
- added U8: 74HC595, Package_SO:SOIC-16_3.9x9.9mm_P1.27mm, F.Cu at (257.2, 122.8)
- C1, C10, C11, C12, C13, C14, C15, C16, C17, C18, C19, C2, C20, C21, C22, C23, C24, C25, C26, C27, C28, C29, C3, C30, C4, C5, C6, C7, C8, C9, D1, D10, D11, D12, D13, D14, D15, D16, D17, D18, D19, D2, D20, D21, D22, D23, D24, D25, D26, D27, D28, D29, D3, D30, D4, D47, D48, D49, D5, D50, D51, D54, D55, D56, D57, D58, D6, D7, D8, D9: moved to B.Cu
- J3, J4: footprint footprint:ffc-6p-adapter -> Connector_PinSocket_2.54mm:PinSocket_2x03_P2.54mm_Vertical
- SW61, SW62: value SW_DP3T -> SW_DPDT_x2; footprint Button_Switch_THT:SW_Slide_SPDT_Angled_CK_OS102011MA1Q -> Connector:FanPinHeader_1x03_P2.54mm_Vertical
- moved C_IN1 321.7 mm to (16.3, 124.5), turned to -90 degrees
- moved R_FB2 311.8 mm to (13.5, 119.8), turned to 90 degrees
- moved R_PD1 311.5 mm to (13.5, 124.6), turned to -90 degrees
- moved R_FB1 310.2 mm to (15.5, 119.8), turned to -90 degrees
- moved D5 302.2 mm to (25.5, 101.5)
- moved D4 296.1 mm to (25.5, 82.5), turned to 180 degrees
- moved D3 290.6 mm to (25.5, 63.5)
- moved LCSC1 287.5 mm to (27.0, 123.5), turned to 180 degrees
- moved U2 286.9 mm to (21.0, 123.5), turned to 180 degrees
- moved D2 286.0 mm to (25.5, 44.5), turned to 180 degrees
- moved L1 283.9 mm to (30.5, 119.0)
- moved R1 283.4 mm to (41.5, 144.0)
- moved D71 282.2 mm to (49.0, 82.0)
- moved D70 281.9 mm to (49.0, 63.0)
- moved D10 278.1 mm to (44.5, 101.5), turned to 180 degrees
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Connections:
- C_OUT2 pad 1: MT3608_5V0_L -> MT3608_5V0_R
- C_OUT2 pad 2: GND_L -> GND_R
- D1 pad 1: CHAR1_L -> Net-(D1-K)
- D1 pad 2: Net-(D1-A) -> ROW0_L
- D10 pad 1: CHAR5_L -> ROW0_L
- D11 pad 1: CHAR0_L -> Net-(D11-K)
- D11 pad 2: Net-(D101-A) -> ROW0_L
- D12 pad 1: CHAR1_L -> ROW0_L
- D13 pad 1: CHAR3_L -> Net-(D13-K)
- D13 pad 2: Net-(D103-A) -> ROW1_L
- D14 pad 1: CHAR4_L -> ROW1_L
- D15 pad 1: CHAR5_L -> Net-(D15-K)
- D15 pad 2: Net-(D105-A) -> ROW1_L
- D16 pad 1: CHAR2_L -> Net-(D16-K)
- D16 pad 2: Net-(D108-A) -> ROW0_L
- D17 pad 1: CHAR4_L -> ROW0_L
- D18 pad 1: CHAR5_L -> Net-(D18-K)
- D18 pad 2: Net-(D110-A) -> ROW1_L
- D19 pad 1: CHAR0_L -> ROW1_L
- D2 pad 1: CHAR2_L -> ROW0_L
- D20 pad 1: CHAR1_L -> ROW1_L
- D21 pad 1: CHAR0_L -> Net-(D21-K)
- D21 pad 2: Net-(D111-A) -> ROW0_L
- D22 pad 1: CHAR1_L -> ROW0_L
- D23 pad 1: CHAR2_L -> Net-(D23-K)
- D23 pad 2: Net-(D113-A) -> ROW1_L
- D24 pad 1: CHAR3_L -> ROW1_L
- D25 pad 1: CHAR5_L -> Net-(D25-K)
- D25 pad 2: Net-(D115-A) -> ROW0_L
- D26 pad 1: CHAR0_L -> Net-(D26-K)
- D26 pad 2: Net-(D116-A) -> ROW0_L
- D27 pad 1: CHAR1_L -> ROW0_L
- D28 pad 1: CHAR2_L -> Net-(D28-K)
- D28 pad 2: Net-(D118-A) -> ROW1_L
- D29 pad 1: CHAR3_L -> ROW1_L
- D3 pad 1: CHAR3_L -> Net-(D3-K)
- D3 pad 2: Net-(D3-A) -> ROW1_L
- D30 pad 1: CHAR4_L -> Net-(D30-K)
- D30 pad 2: Net-(D120-A) -> ROW1_L
- D31 pad 1: CHAR1_R -> Net-(D31-K)
- D31 pad 2: Net-(D121-A) -> ROW0_R
- D32 pad 1: CHAR2_R -> ROW0_R
- D33 pad 1: CHAR3_R -> Net-(D33-K)
- D33 pad 2: Net-(D123-A) -> ROW1_R
- D34 pad 1: CHAR4_R -> ROW1_R
- D35 pad 1: CHAR5_R -> Net-(D35-K)
- D35 pad 2: Net-(D125-A) -> ROW0_R
- D36 pad 1: CHAR0_R -> Net-(D36-K)
- D36 pad 2: Net-(D126-A) -> ROW0_R
- D37 pad 1: CHAR2_R -> ROW0_R
- D38 pad 1: CHAR3_R -> Net-(D38-K)
- D38 pad 2: Net-(D128-A) -> ROW1_R
- D39 pad 1: CHAR4_R -> ROW1_R
- D4 pad 1: CHAR4_L -> ROW1_L
- D40 pad 1: CHAR5_R -> ROW0_R
- D41 pad 1: CHAR0_R -> Net-(D41-K)
- D41 pad 2: Net-(D131-A) -> ROW0_R
- D42 pad 1: CHAR1_R -> ROW0_R
- D43 pad 1: CHAR3_R -> Net-(D43-K)
- D43 pad 2: Net-(D133-A) -> ROW1_R
- D44 pad 1: CHAR4_R -> ROW1_R
- D45 pad 1: CHAR5_R -> Net-(D45-K)
- D45 pad 2: Net-(D135-A) -> ROW1_R
- D46 pad 1: CHAR0_R -> Net-(D46-K)
- D46 pad 2: Net-(D136-A) -> ROW0_R
- D47 pad 1: CHAR1_R -> ROW0_R
- D48 pad 1: CHAR2_R -> Net-(D48-K)
- D48 pad 2: Net-(D138-A) -> ROW1_R
- D49 pad 1: CHAR4_R -> ROW1_R
- D5 pad 1: CHAR5_L -> Net-(D5-K)
- D5 pad 2: Net-(D5-A) -> ROW0_L
- D50 pad 1: CHAR5_R -> ROW1_R
- D51 pad 1: CHAR0_R -> Net-(D51-K)
- D51 pad 2: Net-(D141-A) -> ROW0_R
- D52 pad 1: CHAR1_R -> ROW0_R
- D53 pad 1: CHAR2_R -> Net-(D53-K)
- D53 pad 2: Net-(D143-A) -> ROW1_R
- D54 pad 1: CHAR3_R -> ROW1_R
- D55 pad 1: CHAR5_R -> Net-(D55-K)
- D55 pad 2: Net-(D145-A) -> ROW0_R
- D56 pad 1: CHAR0_R -> Net-(D56-K)
- D56 pad 2: Net-(D146-A) -> ROW0_R
- D57 pad 1: CHAR1_R -> ROW0_R
- D58 pad 1: CHAR2_R -> Net-(D58-K)
- D58 pad 2: Net-(D148-A) -> ROW1_R
- D59 pad 1: CHAR3_R -> ROW1_R
- D6 pad 1: CHAR0_L -> Net-(D6-K)
- D6 pad 2: Net-(D6-A) -> ROW0_L
- D60 pad 1: CHAR4_R -> Net-(D60-K)
- D60 pad 2: Net-(D150-A) -> ROW1_R
- D7 pad 1: CHAR2_L -> ROW0_L
- D8 pad 1: CHAR3_L -> Net-(D8-K)
- D8 pad 2: Net-(D8-A) -> ROW1_L
- D9 pad 1: CHAR4_L -> ROW1_L
- J3 pad 1: TP_VCC_L -> TP_SDA_L
- J3 pad 2: INTR_L -> GND_L
- J3 pad 5: TP_SDA_L -> TP_VCC_L
- J3 pad 6: GND_L -> INTR_L
- J4 pad 1: TP_VCC_R -> TP_SDA_R
- J4 pad 2: INTR_R -> GND_R
- J4 pad 5: TP_SDA_R -> TP_VCC_R
- J4 pad 6: GND_R -> INTR_R
- SW1 pad 1: CHAR0_L -> COL0_L
- SW1 pad 2: Net-(D1-A) -> Net-(D1-K)
- SW10 pad 1: CHAR1_L -> COL6_L
- SW11 pad 1: CHAR2_L -> COL2_L
- SW11 pad 2: Net-(D101-A) -> Net-(D11-K)
- SW12 pad 1: CHAR2_L -> COL2_L
- SW13 pad 1: CHAR2_L -> COL2_L
- SW13 pad 2: Net-(D103-A) -> Net-(D13-K)
- SW14 pad 1: CHAR2_L -> COL2_L
- SW15 pad 1: CHAR2_L -> COL6_L
- SW15 pad 2: Net-(D105-A) -> Net-(D15-K)
- SW16 pad 1: CHAR3_L -> COL3_L
- SW16 pad 2: Net-(D108-A) -> Net-(D16-K)
- SW17 pad 1: CHAR3_L -> COL3_L
- SW18 pad 1: CHAR3_L -> COL3_L
- SW18 pad 2: Net-(D110-A) -> Net-(D18-K)
- SW19 pad 1: CHAR3_L -> COL3_L
- SW2 pad 1: CHAR0_L -> COL0_L
- SW20 pad 1: CHAR3_L -> COL6_L
- SW21 pad 1: CHAR4_L -> COL4_L
- SW21 pad 2: Net-(D111-A) -> Net-(D21-K)
- SW22 pad 1: CHAR4_L -> COL4_L
- SW23 pad 1: CHAR4_L -> COL4_L
- SW23 pad 2: Net-(D113-A) -> Net-(D23-K)
- SW24 pad 1: CHAR4_L -> COL4_L
- SW25 pad 1: CHAR4_L -> COL7_L
- SW25 pad 2: Net-(D115-A) -> Net-(D25-K)
- SW26 pad 1: CHAR5_L -> COL5_L
- SW26 pad 2: Net-(D116-A) -> Net-(D26-K)
- SW27 pad 1: CHAR5_L -> COL5_L
- SW28 pad 1: CHAR5_L -> COL5_L
- SW28 pad 2: Net-(D118-A) -> Net-(D28-K)
- SW29 pad 1: CHAR5_L -> COL5_L
- SW3 pad 1: CHAR0_L -> COL0_L
- SW3 pad 2: Net-(D3-A) -> Net-(D3-K)
- SW30 pad 1: CHAR5_L -> COL7_L
- SW30 pad 2: Net-(D120-A) -> Net-(D30-K)
- SW31 pad 1: CHAR0_R -> COL0_R
- SW31 pad 2: Net-(D121-A) -> Net-(D31-K)
- SW32 pad 1: CHAR0_R -> COL0_R
- SW33 pad 1: CHAR0_R -> COL0_R
- SW33 pad 2: Net-(D123-A) -> Net-(D33-K)
- SW34 pad 1: CHAR0_R -> COL0_R
- SW35 pad 1: CHAR0_R -> COL6_R
- SW35 pad 2: Net-(D125-A) -> Net-(D35-K)
- SW36 pad 1: CHAR1_R -> COL1_R
- SW36 pad 2: Net-(D126-A) -> Net-(D36-K)
- SW37 pad 1: CHAR1_R -> COL1_R
- SW38 pad 1: CHAR1_R -> COL1_R
- SW38 pad 2: Net-(D128-A) -> Net-(D38-K)
- SW39 pad 1: CHAR1_R -> COL1_R
- SW4 pad 1: CHAR0_L -> COL0_L
- SW40 pad 1: CHAR1_R -> COL6_R
- SW41 pad 1: CHAR2_R -> COL2_R
- SW41 pad 2: Net-(D131-A) -> Net-(D41-K)
- SW42 pad 1: CHAR2_R -> COL2_R
- SW43 pad 1: CHAR2_R -> COL2_R
- SW43 pad 2: Net-(D133-A) -> Net-(D43-K)
- SW44 pad 1: CHAR2_R -> COL2_R
- SW45 pad 1: CHAR2_R -> COL6_R
- SW45 pad 2: Net-(D135-A) -> Net-(D45-K)
- SW46 pad 1: CHAR3_R -> COL3_R
- SW46 pad 2: Net-(D136-A) -> Net-(D46-K)
- SW47 pad 1: CHAR3_R -> COL3_R
- SW48 pad 1: CHAR3_R -> COL3_R
- SW48 pad 2: Net-(D138-A) -> Net-(D48-K)
- SW49 pad 1: CHAR3_R -> COL3_R
- SW5 pad 1: CHAR0_L -> COL6_L
- SW5 pad 2: Net-(D5-A) -> Net-(D5-K)
- SW50 pad 1: CHAR3_R -> COL6_R
- SW51 pad 1: CHAR4_R -> COL4_R
- SW51 pad 2: Net-(D141-A) -> Net-(D51-K)
- SW52 pad 1: CHAR4_R -> COL4_R
- SW53 pad 1: CHAR4_R -> COL4_R
- SW53 pad 2: Net-(D143-A) -> Net-(D53-K)
- SW54 pad 1: CHAR4_R -> COL4_R
- SW55 pad 1: CHAR4_R -> COL7_R
- SW55 pad 2: Net-(D145-A) -> Net-(D55-K)
- SW56 pad 1: CHAR5_R -> COL5_R
- SW56 pad 2: Net-(D146-A) -> Net-(D56-K)
- SW57 pad 1: CHAR5_R -> COL5_R
- SW58 pad 1: CHAR5_R -> COL5_R
- SW58 pad 2: Net-(D148-A) -> Net-(D58-K)
- SW59 pad 1: CHAR5_R -> COL5_R
- SW6 pad 1: CHAR1_L -> COL1_L
- SW6 pad 2: Net-(D6-A) -> Net-(D6-K)
- SW60 pad 1: CHAR5_R -> COL7_R
- SW60 pad 2: Net-(D150-A) -> Net-(D60-K)
- SW61 pad 2: unconnected-(SW61-Pad2) -> VBATT_L
- SW61 pad 3: VBATT_L -> unconnected-(SW61A-C-Pad3)
- SW62 pad 1: VBATT_RAW_R -> unconnected-(SW62A-A-Pad1)
- SW62 pad 2: unconnected-(SW62-Pad2) -> VBATT_R
- SW62 pad 3: VBATT_R -> VBATT_RAW_R
- SW7 pad 1: CHAR1_L -> COL1_L
- SW8 pad 1: CHAR1_L -> COL1_L
- SW8 pad 2: Net-(D8-A) -> Net-(D8-K)
- SW9 pad 1: CHAR1_L -> COL1_L
- U1 pad 1: CHAR0_L -> SRCLK_L
- U1 pad 2: CHAR1_L -> RCLK_L
- U1 pad 3: CHAR2_L -> SER_L
- U1 pad 4: CHAR3_L -> ROW0_L
- U1 pad 5: CHAR4_L -> ROW1_L
- U1 pad 6: CHAR5_L -> unconnected-(U1-D5-Pad6)
- U3 pad 4: MT3608_5V0_L -> Net-(U3-PR1)
- U3 pad 5: unconnected-(U3-MODE-Pad5) -> USB_5V0_L
- U4 pad 1: CHAR0_R -> SRCLK_R
- U4 pad 2: CHAR1_R -> RCLK_R
- U4 pad 3: CHAR2_R -> SER_R
- U4 pad 4: CHAR3_R -> ROW0_R
- U4 pad 5: CHAR4_R -> ROW1_R
- U4 pad 6: CHAR5_R -> unconnected-(U4-D5-Pad6)
- U6 pad 4: MT3608_5V0_R -> Net-(U6-PR1)
- U6 pad 5: unconnected-(U6-MODE-Pad5) -> USB_5V0_R
Routing:
- net GND_L: track 0.00 -> 188.8 mm, vias 0 -> 7
- net VBATT_L: track 0.00 -> 186.5 mm
- net VBATT_RAW_L: track 0.00 -> 66.2 mm
- net MT3608_5V0_L: track 0.00 -> 30.2 mm, vias 0 -> 3
- net BST_EN_L: track 0.00 -> 23.8 mm, vias 0 -> 4
- net Net-(LCSC1-A): track 0.00 -> 14.4 mm
- net Net-(U2-FB): track 0.00 -> 10.7 mm, vias 0 -> 2
Other:
- board outline added: 135 x 135 mm

Commit message: mod2
Parts:
- R_PM1, R_PM3: value 30kR -> 10kR
- moved R_DM2 77.7 mm to (21.5, 147.8), turned to -90 degrees
- moved R_DM4 77.3 mm to (24.0, 147.8), turned to -90 degrees
- moved R_PM1 76.6 mm to (19.7, 131.5)
- moved C_PM1 75.3 mm to (15.5, 131.5)
- moved U3 69.8 mm to (35.8, 121.2), turned to -90 degrees
- moved R_PM2 68.8 mm to (35.0, 118.0), turned to 180 degrees
- moved C_PM3 67.9 mm to (39.0, 123.0)
- moved C_PM2 58.1 mm to (37.0, 125.0)
- moved U7 54.2 mm to (51.0, 124.5), turned to -90 degrees
- moved C_SR1 49.7 mm to (44.0, 122.8), turned to 90 degrees
- moved J1 46.2 mm to (52.0, 150.0), turned to 90 degrees
- moved REF** 29.0 mm to (140.0, 150.2)
- moved SW61 28.5 mm to (109.5, 151.0)
- moved D1 12.0 mm to (34.0, 34.0)
- moved D10 12.0 mm to (53.0, 110.0)
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Connections:
- U3 pad 5: USB_5V0_L -> MT3608_5V0_L
- U6 pad 5: USB_5V0_R -> MT3608_5V0_R
Routing:
- net ROW0_L: track 0.00 -> 471.2 mm, vias 0 -> 8
- net LED_5V0_L: track 0.00 -> 397.8 mm, vias 0 -> 16
- net ROW1_L: track 0.00 -> 392.9 mm, vias 0 -> 5
- net GND_L: track 188.8 -> 1.05 mm, vias 7 -> 0
- net COL5_L: track 0.00 -> 171.8 mm, vias 0 -> 10
- net COL4_L: track 0.00 -> 152.3 mm, vias 0 -> 14
- net COL3_L: track 0.00 -> 134.3 mm, vias 0 -> 12
- net COL1_L: track 0.00 -> 124.8 mm, vias 0 -> 8
- net COL0_L: track 0.00 -> 123.8 mm, vias 0 -> 7
- net Net-(D61-DIN): track 0.00 -> 112.1 mm, vias 0 -> 6
- net COL2_L: track 0.00 -> 111.0 mm, vias 0 -> 10
- net TP_VCC_L: track 0.00 -> 92.5 mm, vias 0 -> 3
- net COL7_L: track 0.00 -> 84.5 mm, vias 0 -> 2
- net COL6_L: track 0.00 -> 68.2 mm, vias 0 -> 2
- net INTR_L: track 0.00 -> 67.1 mm, vias 0 -> 1
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
Commit message: mod_pcb_comp
Parts:
- added REF**: MountingHole_2.2mm_M2, MountingHole:MountingHole_2.2mm_M2, F.Cu at (220.5, 140.5)
- added REF**: MountingHole_2.2mm_M2, MountingHole:MountingHole_2.2mm_M2, F.Cu at (220.5, 55.5)
- added REF**: MountingHole_2.2mm_M2, MountingHole:MountingHole_2.2mm_M2, F.Cu at (345.5, 55.5)
- added REF**: MountingHole_2.2mm_M2, MountingHole:MountingHole_2.2mm_M2, F.Cu at (345.5, 140.5)
- added REF**: MountingHole_2.2mm_M2, MountingHole:MountingHole_2.2mm_M2, F.Cu at (345.5, 180.5)
- added REF**: MountingHole_2.2mm_M2, MountingHole:MountingHole_2.2mm_M2, F.Cu at (220.5, 180.5)
- added R_DM1: 10k, Resistor_SMD:R_0603_1608Metric, F.Cu at (82.5, 174.2)
- added R_DM3: 10k, Resistor_SMD:R_0603_1608Metric, F.Cu at (76.8, 174.2)
- added R_DM5: 10k, Resistor_SMD:R_0603_1608Metric, F.Cu at (336.5, 162.3)
- added R_DM6: 10k, Resistor_SMD:R_0603_1608Metric, F.Cu at (334.5, 162.3)
- D31, D32, D33, D34, D35, D36, D37, D38, D39, D40, D41, D42, D43, D44, D45, D46, D52, D53, D59, D60: moved to B.Cu
- moved C26 210.2 mm to (311.5, 112.2)
- moved D50 207.6 mm to (296.5, 140.2)
- moved C16 202.8 mm to (311.5, 74.2)
- moved D55 199.5 mm to (315.5, 140.2), turned to 0 degrees
- moved C25 197.8 mm to (311.5, 93.2)
- moved C27 196.5 mm to (292.5, 112.2)
- moved D49 192.0 mm to (296.5, 121.2)
- moved C17 188.9 mm to (292.5, 74.2)
- moved C24 187.4 mm to (292.5, 93.2)
- moved D45 186.8 mm to (277.5, 140.2)
- moved D60 184.5 mm to (334.5, 140.2)
- moved D54 184.0 mm to (315.5, 121.2)
- moved D40 183.6 mm to (258.5, 140.2), turned to 180 degrees
- moved D35 181.5 mm to (239.5, 140.2)
- moved C28 181.4 mm to (273.5, 112.2)
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Connections:
- C_SR1 pad 2: Net-(U7-GND) -> TP_VCC_L
- C_SR2 pad 2: Net-(U8-GND) -> TP_VCC_R
- U7 pad 8: Net-(U7-GND) -> GND_L
- U8 pad 8: Net-(U8-GND) -> GND_R
Routing:
- net ROW0_R: track 0.00 -> 483.6 mm, vias 0 -> 7
- net LED_5V0_R: track 0.00 -> 414.2 mm, vias 0 -> 18
- net ROW1_R: track 0.00 -> 357.7 mm, vias 0 -> 7
- net VBATT_R: track 0.00 -> 215.5 mm, vias 0 -> 5
- net COL0_R: track 0.00 -> 186.5 mm, vias 0 -> 10
- net COL1_R: track 0.00 -> 158.2 mm, vias 0 -> 12
- net COL2_R: track 0.00 -> 140.1 mm, vias 0 -> 12
- net COL5_R: track 0.00 -> 117.5 mm, vias 0 -> 6
- net COL3_R: track 0.00 -> 114.9 mm, vias 0 -> 10
- net COL6_R: track 0.00 -> 112.7 mm, vias 0 -> 4
- net COL4_R: track 0.00 -> 111.6 mm, vias 0 -> 10
- net Net-(D76-DIN): track 0.00 -> 108.1 mm, vias 0 -> 10
- net TP_VCC_R: track 0.00 -> 88.5 mm, vias 0 -> 4
- net TP_SDA_R: track 0.00 -> 67.1 mm, vias 0 -> 1
- net INTR_R: track 0.00 -> 64.5 mm, vias 0 -> 1
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- added copper zone on B.Cu, net GND_L
- added copper zone on F.Cu, net GND_L
- added copper zone on B.Cu, net GND_R
- added copper zone on F.Cu, net GND_R
Other:
- board size 135 x 135 mm -> 300 x 135.5 mm

Commit message: mod_pcb_order
Changed lines of the file:
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@@
 	)
 	(zone
-		(net "GND_L")
-		(layer "F.Cu")
+		(net "GND_R")
+		(layers "F.Cu" "B.Cu")
 		(hatch edge 0.5)
 		(connect_pads
@@
 		(polygon
 			(pts
-				(xy 187 189) (xy 171.114857 189.828431) (xy 45.5 190.5) (xy 45.5 69.5) (xy 45.43855 47.282284) (xy 147.5 47)
-				(xy 191 47) (xy 196.5 185.5) (xy 195 190)
-			)
-		)
-	)
-	(zone
-		(net "GND_R")
-		(layer "F.Cu")
-		(hatch edge 0.5)
-		(priority 1)
-		(connect_pads
-			(clearance 0.5)
-		)
-		(min_thickness 0.25)
-		(fill yes
-			(thermal_gap 0.5)
-			(thermal_bridge_width 0.5)
-			(island_removal_mode 0)
-		)
-		(polygon
-			(pts
-				(xy 355.489703 45.989073) (xy 355.5 46) (xy 211.5 45.5) (xy 210 187.5) (xy 357 188) (xy 355.5 46)
+				(xy 205.5 37) (xy 212.806551 37.560566) (xy 365 37) (xy 366.263134 193.210578) (xy 205.446368 194.510958)
+				(xy 204 48)
 			)
 		)
@@
 			)
 		)
-	)
-	(zone
-		(net "GND_R")
-		(layer "B.Cu")
-		(hatch edge 0.5)
-		(connect_pads
-			(clearance 0.5)
-		)
-		(min_thickness 0.25)
-		(fill yes
-			(thermal_gap 0.5)
-			(thermal_bridge_width 0.5)
-			(island_removal_mode 0)
-		)
-		(polygon
-			(pts
-				(xy 205.5 37) (xy 212.806551 37.560566) (xy 365 37) (xy 366.263134 193.210578) (xy 205.446368 194.510958)
-				(xy 204 48)
-			)
-		)

Commit message: mod_pcb_order_comp
Parts:
- removed LCSC1, LCSC2: C81579, Diode_SMD:D_SMA
- added D_5B2: SS34, Diode_SMD:D_SMA, F.Cu at (318.5, 149.5)
- added D_5B_1: SS34, Diode_SMD:D_SMA, F.Cu at (67.1, 151.6)
- D61, D62, D63, D64, D65, D66, D67, D68, D69, D70, D71, D72, D73, D74, D75, D76, D77, D78, D79, D80, D81, D82, D83, D84, D85, D86, D87, D88, D89, D90: value WS2812B-2020 -> SK6805-EC20
- REF** (x4): value MountingHole_2.2mm_M2 -> MH2.2mmM2
- moved C16 15.5 mm to (296.0, 73.8)
- moved C17 15.5 mm to (277.0, 73.8)
- moved C18 15.5 mm to (258.0, 73.8)
- moved C19 15.5 mm to (239.0, 73.8)
- moved C20 15.5 mm to (220.0, 73.8)
- moved C21 15.5 mm to (220.0, 92.8)
- moved C22 15.5 mm to (239.0, 92.8)
- moved C23 15.5 mm to (258.0, 92.8)
- moved C24 15.5 mm to (277.0, 92.8)
- moved C25 15.5 mm to (296.0, 92.8)
- moved C26 15.5 mm to (296.0, 111.8)
- moved C27 15.5 mm to (277.0, 111.8)
- moved C28 15.5 mm to (258.0, 111.8)
- moved C29 15.5 mm to (239.0, 111.8)
- moved C30 15.5 mm to (220.0, 111.8)
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Other:
- board size 300 x 135.5 mm -> 285 x 135 mm
- board text added: "User Cut"
