File: pcb/mks_mkb1/mks_mkb1.kicad_pcb (KiCad board)
At the start: 2 copper layers, 285 x 135 mm, 242 parts, among them J1 Conn_01x02, J2 Conn_01x02, J3 Conn_01x06_Pin, J4 Conn_01x06_Pin, SW1 SW_Push, SW10 SW_Push, SW11 SW_Push, SW12 SW_Push, SW13 SW_Push, SW14 SW_Push, SW15 SW_Push, SW16 SW_Push, SW17 SW_Push, SW18 SW_Push, SW19 SW_Push, SW2 SW_Push, SW20 SW_Push, SW21 SW_Push, SW22 SW_Push, SW23 SW_Push, SW24 SW_Push, SW25 SW_Push, SW26 SW_Push, SW27 SW_Push, SW28 SW_Push, SW29 SW_Push, SW3 SW_Push, SW30 SW_Push, SW31 SW_Push, SW32 SW_Push, SW33 SW_Push, SW34 SW_Push, SW35 SW_Push, SW36 SW_Push, SW37 SW_Push, SW38 SW_Push, SW39 SW_Push, SW4 SW_Push, SW40 SW_Push, SW41 SW_Push, SW42 SW_Push, SW43 SW_Push, SW44 SW_Push, SW45 SW_Push, SW46 SW_Push, SW47 SW_Push, SW48 SW_Push, SW49 SW_Push, SW5 SW_Push, SW50 SW_Push, SW51 SW_Push, SW52 SW_Push, SW53 SW_Push, SW54 SW_Push, SW55 SW_Push, SW56 SW_Push, SW57 SW_Push, SW58 SW_Push, SW59 SW_Push, SW6 SW_Push, SW60 SW_Push, SW61 SW_DPDT_x2, SW62 SW_DPDT_x2, SW7 SW_Push, SW8 SW_Push, SW9 SW_Push, U1 XIAO-nRF52840-SMD, U2 MT3608, U3 TPS2116DRL, U4 XIAO-nRF52840-SMD, U5 MT3608, U6 TPS2116DRL, U7 74HC595, U8 74HC595

Commit message: mod_pcb_order_comp
Parts:
- D61, D62, D63, D64, D65, D66, D67, D68, D69, D70, D71, D72, D73, D74, D75, D76, D77, D78, D79, D80, D81, D82, D83, D84, D85, D86, D87, D88, D89, D90: footprint LED_SMD:LED_WS2812B-2020_PLCC4_2.0x2.0mm -> Mks_Library:SK6805-EC20
- moved D61 0.25 mm to (89.0, 74.0)
- moved D62 0.25 mm to (108.0, 74.0), turned to 90 degrees
- moved D63 0.25 mm to (127.0, 74.0), turned to 90 degrees
- moved D64 0.25 mm to (146.0, 74.0), turned to 90 degrees
- moved D65 0.25 mm to (165.0, 74.0), turned to 90 degrees
- moved D66 0.25 mm to (165.0, 93.0), turned to 90 degrees
- moved D67 0.25 mm to (146.0, 93.0), turned to 90 degrees
- moved D68 0.25 mm to (127.0, 93.0), turned to 90 degrees
- moved D69 0.25 mm to (108.0, 93.0), turned to 90 degrees
- moved D70 0.25 mm to (89.0, 93.0), turned to 90 degrees
- moved D71 0.25 mm to (89.0, 112.0), turned to 90 degrees
- moved D72 0.25 mm to (108.0, 112.0), turned to 90 degrees
- moved D73 0.25 mm to (127.0, 112.0), turned to 90 degrees
- moved D74 0.25 mm to (146.0, 112.0), turned to 90 degrees
- moved D75 0.25 mm to (165.0, 112.0), turned to 90 degrees
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Connections:
- D61 pad 1: Net-(D61-DOUT) -> GND_L
- D61 pad 2: GND_L -> Net-(D61-DIN)
- D61 pad 3: Net-(D61-DIN) -> LED_5V0_L
- D61 pad 4: LED_5V0_L -> Net-(D61-DOUT)
- D62 pad 1: Net-(D62-DOUT) -> GND_L
- D62 pad 2: GND_L -> Net-(D61-DOUT)
- D62 pad 3: Net-(D61-DOUT) -> LED_5V0_L
- D62 pad 4: LED_5V0_L -> Net-(D62-DOUT)
- D63 pad 1: Net-(D63-DOUT) -> GND_L
- D63 pad 2: GND_L -> Net-(D62-DOUT)
- D63 pad 3: Net-(D62-DOUT) -> LED_5V0_L
- D63 pad 4: LED_5V0_L -> Net-(D63-DOUT)
- D64 pad 1: Net-(D64-DOUT) -> GND_L
- D64 pad 2: GND_L -> Net-(D63-DOUT)
- D64 pad 3: Net-(D63-DOUT) -> LED_5V0_L
- D64 pad 4: LED_5V0_L -> Net-(D64-DOUT)
- D65 pad 1: Net-(D65-DOUT) -> GND_L
- D65 pad 2: GND_L -> Net-(D64-DOUT)
- D65 pad 3: Net-(D64-DOUT) -> LED_5V0_L
- D65 pad 4: LED_5V0_L -> Net-(D65-DOUT)
- D66 pad 1: Net-(D66-DOUT) -> GND_L
- D66 pad 2: GND_L -> Net-(D65-DOUT)
- D66 pad 3: Net-(D65-DOUT) -> LED_5V0_L
- D66 pad 4: LED_5V0_L -> Net-(D66-DOUT)
- D67 pad 1: Net-(D67-DOUT) -> GND_L
- D67 pad 2: GND_L -> Net-(D66-DOUT)
- D67 pad 3: Net-(D66-DOUT) -> LED_5V0_L
- D67 pad 4: LED_5V0_L -> Net-(D67-DOUT)
- D68 pad 1: Net-(D68-DOUT) -> GND_L
- D68 pad 2: GND_L -> Net-(D67-DOUT)
- D68 pad 3: Net-(D67-DOUT) -> LED_5V0_L
- D68 pad 4: LED_5V0_L -> Net-(D68-DOUT)
- D69 pad 1: Net-(D69-DOUT) -> GND_L
- D69 pad 2: GND_L -> Net-(D68-DOUT)
- D69 pad 3: Net-(D68-DOUT) -> LED_5V0_L
- D69 pad 4: LED_5V0_L -> Net-(D69-DOUT)
- D70 pad 1: Net-(D70-DOUT) -> GND_L
- D70 pad 2: GND_L -> Net-(D69-DOUT)
- D70 pad 3: Net-(D69-DOUT) -> LED_5V0_L
- D70 pad 4: LED_5V0_L -> Net-(D70-DOUT)
- D71 pad 1: Net-(D71-DOUT) -> GND_L
- D71 pad 2: GND_L -> Net-(D70-DOUT)
- D71 pad 3: Net-(D70-DOUT) -> LED_5V0_L
- D71 pad 4: LED_5V0_L -> Net-(D71-DOUT)
- D72 pad 1: Net-(D72-DOUT) -> GND_L
- D72 pad 2: GND_L -> Net-(D71-DOUT)
- D72 pad 3: Net-(D71-DOUT) -> LED_5V0_L
- D72 pad 4: LED_5V0_L -> Net-(D72-DOUT)
- D73 pad 1: Net-(D73-DOUT) -> GND_L
- D73 pad 2: GND_L -> Net-(D72-DOUT)
- D73 pad 3: Net-(D72-DOUT) -> LED_5V0_L
- D73 pad 4: LED_5V0_L -> Net-(D73-DOUT)
- D74 pad 1: Net-(D74-DOUT) -> GND_L
- D74 pad 2: GND_L -> Net-(D73-DOUT)
- D74 pad 3: Net-(D73-DOUT) -> LED_5V0_L
- D74 pad 4: LED_5V0_L -> Net-(D74-DOUT)
- D75 pad 1: unconnected-(D75-DOUT-Pad1) -> GND_L
- D75 pad 2: GND_L -> Net-(D74-DOUT)
- D75 pad 3: Net-(D74-DOUT) -> LED_5V0_L
- D75 pad 4: LED_5V0_L -> unconnected-(D75-DOUT-Pad4)
- D76 pad 1: Net-(D76-DOUT) -> GND_R
- D76 pad 2: GND_R -> Net-(D76-DIN)
- D76 pad 3: Net-(D76-DIN) -> LED_5V0_R
- D76 pad 4: LED_5V0_R -> Net-(D76-DOUT)
- D77 pad 1: Net-(D77-DOUT) -> GND_R
- D77 pad 2: GND_R -> Net-(D76-DOUT)
- D77 pad 3: Net-(D76-DOUT) -> LED_5V0_R
- D77 pad 4: LED_5V0_R -> Net-(D77-DOUT)
- D78 pad 1: Net-(D78-DOUT) -> GND_R
- D78 pad 2: GND_R -> Net-(D77-DOUT)
- D78 pad 3: Net-(D77-DOUT) -> LED_5V0_R
- D78 pad 4: LED_5V0_R -> Net-(D78-DOUT)
- D79 pad 1: Net-(D79-DOUT) -> GND_R
- D79 pad 2: GND_R -> Net-(D78-DOUT)
- D79 pad 3: Net-(D78-DOUT) -> LED_5V0_R
- D79 pad 4: LED_5V0_R -> Net-(D79-DOUT)
- D80 pad 1: Net-(D80-DOUT) -> GND_R
- D80 pad 2: GND_R -> Net-(D79-DOUT)
- D80 pad 3: Net-(D79-DOUT) -> LED_5V0_R
- D80 pad 4: LED_5V0_R -> Net-(D80-DOUT)
- D81 pad 1: Net-(D81-DOUT) -> GND_R
- D81 pad 2: GND_R -> Net-(D80-DOUT)
- D81 pad 3: Net-(D80-DOUT) -> LED_5V0_R
- D81 pad 4: LED_5V0_R -> Net-(D81-DOUT)
- D82 pad 1: Net-(D82-DOUT) -> GND_R
- D82 pad 2: GND_R -> Net-(D81-DOUT)
- D82 pad 3: Net-(D81-DOUT) -> LED_5V0_R
- D82 pad 4: LED_5V0_R -> Net-(D82-DOUT)
- D83 pad 1: Net-(D83-DOUT) -> GND_R
- D83 pad 2: GND_R -> Net-(D82-DOUT)
- D83 pad 3: Net-(D82-DOUT) -> LED_5V0_R
- D83 pad 4: LED_5V0_R -> Net-(D83-DOUT)
- D84 pad 1: Net-(D84-DOUT) -> GND_R
- D84 pad 2: GND_R -> Net-(D83-DOUT)
- D84 pad 3: Net-(D83-DOUT) -> LED_5V0_R
- D84 pad 4: LED_5V0_R -> Net-(D84-DOUT)
- D85 pad 1: Net-(D85-DOUT) -> GND_R
- D85 pad 2: GND_R -> Net-(D84-DOUT)
- D85 pad 3: Net-(D84-DOUT) -> LED_5V0_R
- D85 pad 4: LED_5V0_R -> Net-(D85-DOUT)
- D86 pad 1: Net-(D86-DOUT) -> GND_R
- D86 pad 2: GND_R -> Net-(D85-DOUT)
- D86 pad 3: Net-(D85-DOUT) -> LED_5V0_R
- D86 pad 4: LED_5V0_R -> Net-(D86-DOUT)
- D87 pad 1: Net-(D87-DOUT) -> GND_R
- D87 pad 2: GND_R -> Net-(D86-DOUT)
- D87 pad 3: Net-(D86-DOUT) -> LED_5V0_R
- D87 pad 4: LED_5V0_R -> Net-(D87-DOUT)
- D88 pad 1: Net-(D88-DOUT) -> GND_R
- D88 pad 2: GND_R -> Net-(D87-DOUT)
- D88 pad 3: Net-(D87-DOUT) -> LED_5V0_R
- D88 pad 4: LED_5V0_R -> Net-(D88-DOUT)
- D89 pad 1: Net-(D89-DOUT) -> GND_R
- D89 pad 2: GND_R -> Net-(D88-DOUT)
- D89 pad 3: Net-(D88-DOUT) -> LED_5V0_R
- D89 pad 4: LED_5V0_R -> Net-(D89-DOUT)
- D90 pad 1: unconnected-(D90-DOUT-Pad1) -> GND_R
- D90 pad 2: GND_R -> Net-(D89-DOUT)
- D90 pad 3: Net-(D89-DOUT) -> LED_5V0_R
- D90 pad 4: LED_5V0_R -> unconnected-(D90-DOUT-Pad4)
Routing:
- net GND_R: track 22.9 -> 30.5 mm
- net Net-(D61-DOUT): track 32.4 -> 27.6 mm
- net Net-(D61-DIN): track 119.1 -> 116.5 mm
- net LED_5V0_R: track 414.2 -> 415.9 mm
- net Net-(D62-DOUT): track 32.3 -> 30.8 mm
- net GND_L: track 16.9 -> 18.3 mm, vias 13 -> 15
- net Net-(D65-DOUT): track 34.5 -> 35.4 mm
- net Net-(D67-DOUT): track 19.7 -> 20.5 mm
- net Net-(D84-DOUT): track 33.4 -> 34.2 mm
- net Net-(D77-DOUT): track 19.0 -> 19.8 mm
- net Net-(D72-DOUT): track 31.2 -> 32.0 mm
- net Net-(D71-DOUT): track 31.2 -> 32.0 mm
- net Net-(D70-DOUT): track 28.1 -> 28.8 mm
- net Net-(D69-DOUT): track 19.7 -> 20.5 mm
- net Net-(D68-DOUT): track 19.7 -> 20.5 mm
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