File: pcb/mks_mkb1/mks_mkb1.kicad_sch (KiCad schematic)
At the start: 272 parts, among them J1 Conn_01x02, J2 Conn_01x02, J3 Conn_01x06_Pin, J4 Conn_01x06_Pin, SW1 SW_Push, SW10 SW_Push, SW11 SW_Push, SW12 SW_Push, SW13 SW_Push, SW14 SW_Push, SW15 SW_Push, SW16 SW_Push, SW17 SW_Push, SW18 SW_Push, SW19 SW_Push, SW2 SW_Push, SW20 SW_Push, SW21 SW_Push, SW22 SW_Push, SW23 SW_Push, SW24 SW_Push, SW25 SW_Push, SW26 SW_Push, SW27 SW_Push, SW28 SW_Push, SW29 SW_Push, SW3 SW_Push, SW30 SW_Push, SW31 SW_Push, SW32 SW_Push, SW33 SW_Push, SW34 SW_Push, SW35 SW_Push, SW36 SW_Push, SW37 SW_Push, SW38 SW_Push, SW39 SW_Push, SW4 SW_Push, SW40 SW_Push, SW41 SW_Push, SW42 SW_Push, SW43 SW_Push, SW44 SW_Push, SW45 SW_Push, SW46 SW_Push, SW47 SW_Push, SW48 SW_Push, SW49 SW_Push, SW5 SW_Push, SW50 SW_Push, SW51 SW_Push, SW52 SW_Push, SW53 SW_Push, SW54 SW_Push, SW55 SW_Push, SW56 SW_Push, SW57 SW_Push, SW58 SW_Push, SW59 SW_Push, SW6 SW_Push, SW60 SW_Push, SW61 SW_DP3T, SW62 SW_DP3T, SW7 SW_Push, SW8 SW_Push, SW9 SW_Push, U1 XIAO-nRF52840-SMD, U2 MT3608, U3 TPS2116DRL, U4 XIAO-nRF52840-SMD, U5 MT3608, U6 TPS2116DRL

Commit message: mod1
Parts:
- removed D100, D101, D102, D103, D104, D105, D106, D107, D108, D109, D110, D111, D112, D113, D114, D115, D116, D117, D118, D119, D120, D121, D122, D123, D124, D125, D126, D127, D128, D129, D130, D131, D132, D133, D134, D135, D136, D137, D138, D139, D140, D141, D142, D143, D144, D145, D146, D147, D148, D149, D150, D91, D92, D93, D94, D95, D96, D97, D98, D99: D, Diode_SMD:D_SOD-123, symbol Device:D
- removed R5: 39kR, Resistor_SMD:R_0603_1608Metric, symbol Device:R
- removed R6: 10kR, Resistor_SMD:R_0603_1608Metric, symbol Device:R
- removed SW61, SW62: SW_DP3T, Button_Switch_THT:SW_Slide_SPDT_Angled_CK_OS102011MA1Q, symbol Switch:SW_DP3T
- added C_PM1, C_PM2, C_PM4, C_PM5: 4.7µF, Capacitor_SMD:C_0603_1608Metric, symbol Device:C
- added C_PM3, C_PM6: 47µF, Capacitor_SMD:C_0603_1608Metric, symbol Device:C
- added C_SR1, C_SR2: 0.1µF, Capacitor_SMD:C_0603_1608Metric, symbol Device:C
- added R_DM1, R_DM2, R_DM3, R_DM4, R_DM5, R_DM6, R_DM7, R_DM8: 10k, Resistor_SMD:R_0603_1608Metric, symbol Device:R
- added R_PM3: 30kR, Resistor_SMD:R_0603_1608Metric, symbol Device:R
- added R_PM4: 10kR, Resistor_SMD:R_0603_1608Metric, symbol Device:R
- added SW61, SW62: SW_DPDT_x2, symbol Switch:SW_DPDT_x2
- added U7, U8: 74HC595, Package_SO:SOIC-16_3.9x9.9mm_P1.27mm, symbol 74xx:74HC595
- J3, J4: footprint footprint:ffc-6p-adapter -> Connector_PinSocket_2.54mm:PinSocket_2x03_P2.54mm_Vertical
- R_PM1: renamed from R2; value 39kR -> 30kR
- renumbered C_OUT2 to C_OUT1, C_OUT3 to C_OUT2, R3 to R_PM2
Connections:
- net GND_L: now also J3.2 (Pin_2), C_PM1.2, C_PM2.2, C_PM3.2, C_SR1.1, R_DM2.2, R_DM4.2, U7.13 (~{OE}); no longer J3.6 (Pin_6)
- net GND_R: now also J4.2 (Pin_2), C_PM4.2, C_PM5.2, C_PM6.2, C_SR2.1, R_DM7.2, R_DM8.2, R_PM4.1, U8.13 (~{OE}); no longer J4.6 (Pin_6)
- net INTR_L: now also J3.6 (Pin_6); no longer J3.2 (Pin_2)
- net INTR_R: now also J4.6 (Pin_6); no longer J4.2 (Pin_2)
- net LED_5V0_L: now also C_PM3.1
- net LED_5V0_R: now also C_PM6.1
- net MT3608_5V0_L: now also C_PM2.1; no longer R_PM1.2, R_PM2.2, U3.4 (PR1)
- net MT3608_5V0_R: now also C_PM5.1; no longer U6.4 (PR1)
- net TP_SDA_L: now also J3.1 (Pin_1); no longer J3.5 (Pin_5)
- net TP_SDA_R: now also J4.1 (Pin_1); no longer J4.5 (Pin_5)
- net TP_VCC_L: now also J3.5 (Pin_5), R_DM1.2, R_DM3.2, U7.16 (VCC); no longer J3.1 (Pin_1)
- net TP_VCC_R: now also J4.5 (Pin_5), R_DM5.2, R_DM6.2, U8.16 (VCC); no longer J4.1 (Pin_1)
- net USB_5V0_L: now also U3.5 (MODE), C_PM1.1
- net USB_5V0_R: now also U6.5 (MODE), C_PM4.1, R_PM3.1
- net VBATT_L: now also SW61.2 (B)
- net VBATT_R: now also SW62.2 (B)
- net VBATT_RAW_L: now also SW61.1 (A)
- net VBATT_RAW_R: now also SW62.3 (C)
- net at SW36.2: now also D36.1 (K); no longer D36.2 (A)
- net at SW58.2: now also D58.1 (K); no longer D58.2 (A)
- net at SW33.2: now also D33.1 (K); no longer D33.2 (A)
- net at SW31.2: now also D31.1 (K); no longer D31.2 (A)
- net at SW1.2: now also D1.1 (K); no longer D1.2 (A)
- net at SW43.2: now also D43.1 (K); no longer D43.2 (A)
- net at SW3.2: now also D3.1 (K); no longer D3.2 (A)
- net at SW13.2: now also D13.1 (K); no longer D13.2 (A)
- net at SW30.2: now also D30.1 (K); no longer D30.2 (A)
- net at SW51.2: now also D51.1 (K); no longer D51.2 (A)
- net at SW5.2: now also D5.1 (K); no longer D5.2 (A)
- net at SW15.2: now also D15.1 (K); no longer D15.2 (A)
- net at SW53.2: now also D53.1 (K); no longer D53.2 (A)
- net at SW21.2: now also D21.1 (K); no longer D21.2 (A)
- net at SW18.2: now also D18.1 (K); no longer D18.2 (A)
- net at SW46.2: now also D46.1 (K); no longer D46.2 (A)
- net at SW11.2: now also D11.1 (K); no longer D11.2 (A)
- net at SW48.2: now also D48.1 (K); no longer D48.2 (A)
- net at SW35.2: now also D35.1 (K); no longer D35.2 (A)
- net at SW60.2: now also D60.1 (K); no longer D60.2 (A)
- net at SW26.2: now also D26.1 (K); no longer D26.2 (A)
- net at SW6.2: now also D6.1 (K); no longer D6.2 (A)
- net at SW55.2: now also D55.1 (K); no longer D55.2 (A)
- net at SW41.2: now also D41.1 (K); no longer D41.2 (A)
- net at SW38.2: now also D38.1 (K); no longer D38.2 (A)
- net at SW56.2: now also D56.1 (K); no longer D56.2 (A)
- net at SW25.2: now also D25.1 (K); no longer D25.2 (A)
- net at SW45.2: now also D45.1 (K); no longer D45.2 (A)
- net at SW23.2: now also D23.1 (K); no longer D23.2 (A)
- net at SW28.2: now also D28.1 (K); no longer D28.2 (A)
- net at SW16.2: now also D16.1 (K); no longer D16.2 (A)
- net at SW8.2: now also D8.1 (K); no longer D8.2 (A)
- removed net CHAR0_L: D11.1 (K), D19.1 (K), D21.1 (K), D26.1 (K), D6.1 (K), SW1.1, SW2.1, SW3.1, SW4.1, SW5.1, U1.1 (D0)
- removed net CHAR0_R: D36.1 (K), D41.1 (K), D46.1 (K), D51.1 (K), D56.1 (K), SW31.1, SW32.1, SW33.1, SW34.1, SW35.1, U4.1 (D0)
- removed net CHAR1_L: D1.1 (K), D12.1 (K), D20.1 (K), D22.1 (K), D27.1 (K), SW10.1, SW6.1, SW7.1, SW8.1, SW9.1, U1.2 (D1)
- removed net CHAR1_R: D31.1 (K), D42.1 (K), D47.1 (K), D52.1 (K), D57.1 (K), SW36.1, SW37.1, SW38.1, SW39.1, SW40.1, U4.2 (D1)
- removed net CHAR2_L: D16.1 (K), D2.1 (K), D23.1 (K), D28.1 (K), D7.1 (K), SW11.1, SW12.1, SW13.1, SW14.1, SW15.1, U1.3 (D2)
- removed net CHAR2_R: D32.1 (K), D37.1 (K), D48.1 (K), D53.1 (K), D58.1 (K), SW41.1, SW42.1, SW43.1, SW44.1, SW45.1, U4.3 (D2)
- removed net CHAR3_L: D13.1 (K), D24.1 (K), D29.1 (K), D3.1 (K), D8.1 (K), SW16.1, SW17.1, SW18.1, SW19.1, SW20.1, U1.4 (D3)
- removed net CHAR3_R: D33.1 (K), D38.1 (K), D43.1 (K), D54.1 (K), D59.1 (K), SW46.1, SW47.1, SW48.1, SW49.1, SW50.1, U4.4 (D3)
- removed net CHAR4_L: D14.1 (K), D17.1 (K), D30.1 (K), D4.1 (K), D9.1 (K), SW21.1, SW22.1, SW23.1, SW24.1, SW25.1, U1.5 (D4)
- removed net CHAR4_R: D34.1 (K), D39.1 (K), D44.1 (K), D49.1 (K), D60.1 (K), SW51.1, SW52.1, SW53.1, SW54.1, SW55.1, U4.5 (D4)
- removed net CHAR5_L: D10.1 (K), D15.1 (K), D18.1 (K), D25.1 (K), D5.1 (K), SW26.1, SW27.1, SW28.1, SW29.1, SW30.1, U1.6 (D5)
- removed net CHAR5_R: D35.1 (K), D40.1 (K), D45.1 (K), D50.1 (K), D55.1 (K), SW56.1, SW57.1, SW58.1, SW59.1, SW60.1, U4.6 (D5)
- new net: C_SR1.2, U7.8 (GND)
- new net: R_PM1.2, R_PM2.2, U3.4 (PR1)
- new net: R_PM3.2, R_PM4.2, U6.4 (PR1)
- new net: C_SR2.2, U8.8 (GND)
- new net COL0_L: SW1.1, SW2.1, SW3.1, SW4.1, U7.15 (QA)
- new net COL0_R: SW31.1, SW32.1, SW33.1, SW34.1, U8.15 (QA)
- new net COL1_L: SW6.1, SW7.1, SW8.1, SW9.1, U7.1 (QB)
- new net COL1_R: SW36.1, SW37.1, SW38.1, SW39.1, U8.1 (QB)
- new net COL2_L: SW11.1, SW12.1, SW13.1, SW14.1, U7.2 (QC)
- new net COL2_R: SW41.1, SW42.1, SW43.1, SW44.1, U8.2 (QC)
- new net COL3_L: SW16.1, SW17.1, SW18.1, SW19.1, U7.3 (QD)
- new net COL3_R: SW46.1, SW47.1, SW48.1, SW49.1, U8.3 (QD)
- new net COL4_L: SW21.1, SW22.1, SW23.1, SW24.1, U7.4 (QE)
- new net COL4_R: SW51.1, SW52.1, SW53.1, SW54.1, U8.4 (QE)
- new net COL5_L: SW26.1, SW27.1, SW28.1, SW29.1, U7.5 (QF)
- new net COL5_R: SW56.1, SW57.1, SW58.1, SW59.1, U8.5 (QF)
- new net COL6_L: SW10.1, SW15.1, SW20.1, SW5.1, U7.6 (QG)
- new net COL6_R: SW35.1, SW40.1, SW45.1, SW50.1, U8.6 (QG)
- new net COL7_L: SW25.1, SW30.1, U7.7 (QH)
- new net COL7_R: SW55.1, SW60.1, U8.7 (QH)
- new net RCLK_L: U1.2 (D1), U7.12 (RCLK)
- new net RCLK_R: U4.2 (D1), U8.12 (RCLK)
- new net ROW0_L: D1.2 (A), D10.1 (K), D11.2 (A), D12.1 (K), D16.2 (A), D17.1 (K), D2.1 (K), D21.2 (A), D22.1 (K), D25.2 (A), D26.2 (A), D27.1 (K), D5.2 (A), D6.2 (A), D7.1 (K), R_DM1.1, R_DM2.1, U1.4 (D3)
- new net ROW0_R: D31.2 (A), D32.1 (K), D35.2 (A), D36.2 (A), D37.1 (K), D40.1 (K), D41.2 (A), D42.1 (K), D46.2 (A), D47.1 (K), D51.2 (A), D52.1 (K), D55.2 (A), D56.2 (A), D57.1 (K), R_DM5.1, R_DM7.1, U4.4 (D3)
- new net ROW1_L: D13.2 (A), D14.1 (K), D15.2 (A), D18.2 (A), D19.1 (K), D20.1 (K), D23.2 (A), D24.1 (K), D28.2 (A), D29.1 (K), D3.2 (A), D30.2 (A), D4.1 (K), D8.2 (A), D9.1 (K), R_DM3.1, R_DM4.1, U1.5 (D4)
- new net ROW1_R: D33.2 (A), D34.1 (K), D38.2 (A), D39.1 (K), D43.2 (A), D44.1 (K), D45.2 (A), D48.2 (A), D49.1 (K), D50.1 (K), D53.2 (A), D54.1 (K), D58.2 (A), D59.1 (K), D60.2 (A), R_DM6.1, R_DM8.1, U4.5 (D4)
- new net SER_L: U1.3 (D2), U7.14 (SER)
- new net SER_R: U4.3 (D2), U8.14 (SER)
- new net SRCLK_L: U1.1 (D0), U7.11 (SRCLK)
- new net SRCLK_R: U4.1 (D0), U8.11 (SRCLK)
- no-connect marks 22 -> 24
Other:
- note added: "DUPLEX MATRIX"
- note removed: "LOW POWER IMPROVED SQUARE MATRIX"
- moved on the sheet: C1, C10, C11, C12, C13, C14, C15, C16, C17, C18, C19, C2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

Commit message: mod2
Parts:
- R_PM1, R_PM3: value 30kR -> 10kR
Connections:
- net MT3608_5V0_L: now also U3.5 (MODE)
- net MT3608_5V0_R: now also U6.5 (MODE)
- net USB_5V0_L: no longer U3.5 (MODE)
- net USB_5V0_R: no longer U6.5 (MODE)
Changed lines of the file:
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@@
 	)
 	(junction
+		(at 337.82 29.21)
+		(diameter 0)
+		(color 0 0 0 0)
+	)
+	(junction
 		(at 204.47 227.33)
 		(diameter 0)
@@
 	)
 	(junction
-		(at 337.82 29.21)
-		(diameter 0)
-		(color 0 0 0 0)
-	)
-	(junction
 		(at 323.85 54.61)
 		(diameter 0)
@@
 	)
 	(junction
+		(at 332.74 39.37)
+		(diameter 0)
+		(color 0 0 0 0)
+	)
+	(junction
 		(at 229.87 468.63)
 		(diameter 0)
@@
 	)
 	(junction
+		(at 334.01 279.4)
+		(diameter 0)
+		(color 0 0 0 0)
+	)
+	(junction
 		(at 44.45 227.33)
 		(diameter 0)
@@
 	(wire
 		(pts
-			(xy 337.82 36.83) (xy 337.82 29.21)
-		)
-		(stroke
-			(width 0)
-			(type default)
-		)
-	)
-	(wire
-		(pts
 			(xy 232.41 280.67) (xy 245.11 280.67)
 		)
@@
 	(wire
 		(pts
-			(xy 340.36 36.83) (xy 337.82 36.83)
-		)
-		(stroke
-			(width 0)
-			(type default)
-		)
-	)
-	(wire
-		(pts
 			(xy 191.77 336.55) (xy 191.77 345.44)
 		)
@@
 	(wire
 		(pts
-			(xy 339.09 276.86) (xy 339.09 269.24)
-		)
-		(stroke
-			(width 0)
-			(type default)
-		)
-	)
-	(wire
-		(pts
 			(xy 30.48 196.85) (xy 44.45 196.85)
 		)
@@
 	(wire
 		(pts
+			(xy 334.01 279.4) (xy 341.63 279.4)
+		)
+		(stroke
+			(width 0)
+			(type default)
+		)
+	)
+	(wire
+		(pts
 			(xy 326.39 212.09) (xy 334.01 212.09)
 		)
@@
 	(wire
 		(pts
+			(xy 334.01 276.86) (xy 341.63 276.86)
+		)
+		(stroke
+			(width 0)
+			(type default)
+		)
+	)
+	(wire
+		(pts
 			(xy 25.4 290.83) (xy 29.21 290.83)
 		)
@@
 	(wire
 		(pts
-			(xy 337.82 29.21) (xy 340.36 29.21)
+			(xy 326.39 29.21) (xy 337.82 29.21)
 		)
 		(stroke
@@
 	(wire
 		(pts
+			(xy 332.74 39.37) (xy 340.36 39.37)
+		)
+		(stroke
+			(width 0)
+			(type default)
+		)
+	)
+	(wire
+		(pts
 			(xy 184.15 443.23) (xy 184.15 445.77)
 		)
@@
 	(wire
 		(pts
-			(xy 326.39 29.21) (xy 337.82 29.21)
-		)
-		(stroke
-			(width 0)
-			(type default)
-		)
-	)
-	(wire
-		(pts
 			(xy 139.7 269.24) (xy 140.97 269.24)
 		)
@@
 	(wire
 		(pts
+			(xy 332.74 36.83) (xy 340.36 36.83)
+		)
+		(stroke
+			(width 0)
+			(type default)
+		)
+	)
+	(wire
+		(pts
 			(xy 195.58 264.16) (xy 203.2 264.16)
 		)
@@
 	(wire
 		(pts
+			(xy 332.74 36.83) (xy 332.74 39.37)
+		)
+		(stroke
+			(width 0)
+			(type default)
+		)
+	)
+	(wire
+		(pts
 			(xy 113.03 196.85) (xy 113.03 201.93)
 		)
@@
 	(wire
 		(pts
-			(xy 330.2 279.4) (xy 341.63 279.4)
+			(xy 330.2 279.4) (xy 334.01 279.4)
 		)
 		(stroke
@@
 	(wire
 		(pts
-			(xy 341.63 276.86) (xy 339.09 276.86)
-		)
-		(stroke
-			(width 0)
-			(type default)
-		)
-	)
-	(wire
-		(pts
 			(xy 135.89 201.93) (xy 135.89 204.47)
 		)
@@
 	(wire
 		(pts
+			(xy 337.82 29.21) (xy 340.36 29.21)
+		)
+		(stroke
+			(width 0)
+			(type default)
+		)
+	)
+	(wire
+		(pts
 			(xy 168.91 453.39) (xy 176.53 453.39)
 		)
@@
 	(wire
 		(pts
+			(xy 334.01 276.86) (xy 334.01 279.4)
+		)
+		(stroke
+			(width 0)
+			(type default)
+		)
+	)
+	(wire
+		(pts
 			(xy 321.31 438.15) (xy 321.31 443.23)
 		)
@@
 	(wire
 		(pts
-			(xy 328.93 39.37) (xy 340.36 39.37)
+			(xy 328.93 39.37) (xy 332.74 39.37)
 		)
 		(stroke
@@
 			)
 		)
-		(property "Value" "30kR"
+		(property "Value" "10kR"
 			(at 331.47 267.97 90)
 			(show_name no)
@@
 	)
 	(symbol
-		(lib_id "power:PWR_FLAG")
-		(at 337.82 29.21 0)
-		(unit 1)
-		(body_style 1)
-		(exclude_from_sim no)
-		(in_bom yes)
-		(on_board yes)
-		(in_pos_files yes)
-		(dnp no)
-		(property "Reference" "#FLG04"
-			(at 337.82 27.305 0)
-			(hide yes)
-			(show_name no)
-			(do_not_autoplace no)
-			(effects
-				(font
-					(size 1.27 1.27)
-				)
-			)
-		)
-		(property "Value" "PWR_FLAG"
-			(at 337.82 24.638 0)
-			(show_name no)
-			(do_not_autoplace no)
-			(effects
-				(font
-					(size 1.27 1.27)
-				)
-			)
-		)
-		(property "Footprint" ""
-			(at 337.82 29.21 0)
-			(hide yes)
-			(show_name no)
-			(do_not_autoplace no)
-			(effects
-				(font
-					(size 1.27 1.27)
-				)
-			)
-		)
-		(property "Datasheet" ""
-			(at 337.82 29.21 0)
-			(hide yes)
-			(show_name no)
-			(do_not_autoplace no)
-			(effects
-				(font
-					(size 1.27 1.27)
-				)
-			)
-		)
-		(property "Description" "Special symbol for telling ERC where power comes from"
-			(at 337.82 29.21 0)
-			(hide yes)
-			(show_name no)
-			(do_not_autoplace no)
-			(effects
-				(font
-					(size 1.27 1.27)
-				)
-			)
-		)
-		(pin "1"
-		)
-		(instances
-			(project "mks_mkb1"
-				(path "/a01110a3-a326-4798-a058-407730985a8f"
-					(reference "#FLG04")
-					(unit 1)
-				)
-			)
-		)
-	)
-	(symbol
 		(lib_id "Device:D")
 		(at 172.72 147.32 270)
@@
 	)
 	(symbol
+		(lib_id "power:PWR_FLAG")
+		(at 337.82 29.21 0)
+		(unit 1)
+		(body_style 1)
+		(exclude_from_sim no)
+		(in_bom yes)
+		(on_board yes)
+		(in_pos_files yes)
+		(dnp no)
+		(property "Reference" "#FLG010"
+			(at 337.82 27.305 0)
+			(hide yes)
+			(show_name no)
+			(do_not_autoplace no)
+			(effects
+				(font
+					(size 1.27 1.27)
+				)
+			)
+		)
+		(property "Value" "PWR_FLAG"
+			(at 337.82 24.892 0)
+			(show_name no)
+			(do_not_autoplace no)
+			(effects
+				(font
+					(size 1.27 1.27)
+				)
+			)
+		)
+		(property "Footprint" ""
+			(at 337.82 29.21 0)
+			(hide yes)
+			(show_name no)
+			(do_not_autoplace no)
+			(effects
+				(font
+					(size 1.27 1.27)
+				)
+			)
+		)
+		(property "Datasheet" ""
+			(at 337.82 29.21 0)
+			(hide yes)
+			(show_name no)
+			(do_not_autoplace no)
+			(effects
+				(font
+					(size 1.27 1.27)
+				)
+			)
+		)
+		(property "Description" "Special symbol for telling ERC where power comes from"
+			(at 337.82 29.21 0)
+			(hide yes)
+			(show_name no)
+			(do_not_autoplace no)
+			(effects
+				(font
+					(size 1.27 1.27)
+				)
+			)
+		)
+		(pin "1"
+		)
+		(instances
+			(project "mks_mkb1"
+				(path "/a01110a3-a326-4798-a058-407730985a8f"
+					(reference "#FLG010")
+					(unit 1)
+				)
+			)
+		)
+	)
+	(symbol
 		(lib_id "Switch:SW_Push")
 		(at 213.36 162.56 0)
@@
 			)
 		)
-		(property "Value" "30kR"
+		(property "Value" "10kR"
 			(at 330.2 27.94 90)
 			(show_name no)

Commit message: mod_pcb_comp
Connections:
- net GND_L: now also U7.8 (GND)
- net GND_R: now also U8.8 (GND)
- net TP_VCC_L: now also C_SR1.2
- net TP_VCC_R: now also C_SR2.2
Other:
- moved on the sheet: C_SR1, C_SR2

Commit message: mod_pcb_order_comp
Parts:
- C1, C10, C11, C12, C13, C14, C15, C16, C17, C18, C19, C2, C20, C21, C22, C23, C24, C25, C26, C27, C28, C29, C3, C30, C4, C5, C6, C7, C8, C9, C_SR1, C_SR2: LCSC (none) -> C14663
- C_IN1, C_IN2, C_OUT1, C_OUT2: LCSC (none) -> C45783
- C_PM1, C_PM2, C_PM4, C_PM5: LCSC (none) -> C19666
- C_PM3, C_PM6: LCSC (none) -> C15852
- D1, D10, D11, D12, D13, D14, D15, D16, D17, D18, D19, D2, D20, D21, D22, D23, D24, D25, D26, D27, D28, D29, D3, D30, D31, D32, D33, D34, D35, D36, D37, D38, D39, D4, D40, D41, D42, D43, D44, D45, D46, D47, D48, D49, D5, D50, D51, D52, D53, D54, D55, D56, D57, D58, D59, D6, D60, D7, D8, D9: LCSC (none) -> C81598
- D61, D62, D63, D64, D65, D66, D67, D68, D69, D70, D71, D72, D73, D74, D75, D76, D77, D78, D79, D80, D81, D82, D83, D84, D85, D86, D87, D88, D89, D90: value WS2812B-2020 -> SK6805-EC20
- D_5B2: renamed from LCSC2; value C81579 -> SS34
- D_5B_1: renamed from LCSC1; value C81579 -> SS34
- R1, R4: LCSC (none) -> C23138
- R_DM1, R_DM2, R_DM3, R_DM4, R_DM5, R_DM6, R_DM7, R_DM8, R_PM1, R_PM2, R_PM3, R_PM4: LCSC (none) -> C25804
- R_FB1, R_FB3: LCSC (none) -> C23234
- R_FB2, R_FB4: LCSC (none) -> C21190
- R_PD1, R_PD2: LCSC (none) -> C25803

Commit message: mod_pcb_order_comp
Parts:
- removed D61, D62, D63, D64, D65, D66, D67, D68, D69, D70, D71, D72, D73, D74, D75, D76, D77, D78, D79, D80, D81, D82, D83, D84, D85, D86, D87, D88, D89, D90: SK6805-EC20, LED_SMD:LED_WS2812B-2020_PLCC4_2.0x2.0mm, symbol LED:WS2812B-2020
- added D61, D62, D63, D64, D65, D66, D67, D68, D69, D70, D71, D72, D73, D74, D75, D76, D77, D78, D79, D80, D81, D82, D83, D84, D85, D86, D87, D88, D89, D90: SK6805-EC20, Mks_Library:SK6805-EC20, symbol LED:SK6805
Connections:
- net GND_L: now also D61.1 (VSS), D62.1 (VSS), D63.1 (VSS), D64.1 (VSS), D65.1 (VSS), D66.1 (VSS), D67.1 (VSS), D68.1 (VSS), D69.1 (VSS), D70.1 (VSS), D71.1 (VSS), D72.1 (VSS), D73.1 (VSS), D74.1 (VSS), D75.1 (VSS)
- net GND_R: now also D76.1 (VSS), D77.1 (VSS), D78.1 (VSS), D79.1 (VSS), D80.1 (VSS), D81.1 (VSS), D82.1 (VSS), D83.1 (VSS), D84.1 (VSS), D85.1 (VSS), D86.1 (VSS), D87.1 (VSS), D88.1 (VSS), D89.1 (VSS), D90.1 (VSS)
- net LED_5V0_L: now also D61.3 (VDD), D62.3 (VDD), D63.3 (VDD), D64.3 (VDD), D65.3 (VDD), D66.3 (VDD), D67.3 (VDD), D68.3 (VDD), D69.3 (VDD), D70.3 (VDD), D71.3 (VDD), D72.3 (VDD), D73.3 (VDD), D74.3 (VDD), D75.3 (VDD)
- net LED_5V0_R: now also D76.3 (VDD), D77.3 (VDD), D78.3 (VDD), D79.3 (VDD), D80.3 (VDD), D81.3 (VDD), D82.3 (VDD), D83.3 (VDD), D84.3 (VDD), D85.3 (VDD), D86.3 (VDD), D87.3 (VDD), D88.3 (VDD), D89.3 (VDD), D90.3 (VDD)
- net at R4.2: now also D76.2 (DIN)
- net at R1.2: now also D61.2 (DIN)
- new net: D61.4 (DOUT), D62.2 (DIN)
- new net: D79.4 (DOUT), D80.2 (DIN)
- new net: D80.4 (DOUT), D81.2 (DIN)
- new net: D88.4 (DOUT), D89.2 (DIN)
- new net: D89.4 (DOUT), D90.2 (DIN)
- new net: D86.4 (DOUT), D87.2 (DIN)
- new net: D87.4 (DOUT), D88.2 (DIN)
- new net: D67.4 (DOUT), D68.2 (DIN)
- new net: D68.4 (DOUT), D69.2 (DIN)
- new net: D76.4 (DOUT), D77.2 (DIN)
- new net: D77.4 (DOUT), D78.2 (DIN)
- new net: D70.4 (DOUT), D71.2 (DIN)
- new net: D71.4 (DOUT), D72.2 (DIN)
- new net: D69.4 (DOUT), D70.2 (DIN)
- new net: D78.4 (DOUT), D79.2 (DIN)
- new net: D84.4 (DOUT), D85.2 (DIN)
- new net: D85.4 (DOUT), D86.2 (DIN)
- new net: D83.4 (DOUT), D84.2 (DIN)
- new net: D73.4 (DOUT), D74.2 (DIN)
- new net: D74.4 (DOUT), D75.2 (DIN)
- new net: D62.4 (DOUT), D63.2 (DIN)
- new net: D63.4 (DOUT), D64.2 (DIN)
- new net: D65.4 (DOUT), D66.2 (DIN)
- new net: D66.4 (DOUT), D67.2 (DIN)
- new net: D81.4 (DOUT), D82.2 (DIN)
- new net: D72.4 (DOUT), D73.2 (DIN)
- new net: D82.4 (DOUT), D83.2 (DIN)
- new net: D64.4 (DOUT), D65.2 (DIN)
